Commit message: Add integrated QiangNao hands to Kuavo S56

File: src/kuavo_isaaclab_scene/assets/kuavo_s56/urdf/kuavo_s56.urdf (robot description, URDF)
Before this commit: robot biped_s56, 50 links, 49 joints
Links:
- added link l_index_dist, mass 0.011; collision mesh filename=../meshes/l_index_dist.STL; visual mesh filename=../meshes/l_index_dist.STL
- added link l_index_prox, mass 0.008; collision mesh filename=../meshes/l_index_prox.STL; visual mesh filename=../meshes/l_index_prox.STL
- added link l_little_dist, mass 0.008; collision mesh filename=../meshes/l_little_dist.STL; visual mesh filename=../meshes/l_little_dist.STL
- added link l_little_prox, mass 0.008; collision mesh filename=../meshes/l_little_prox.STL; visual mesh filename=../meshes/l_little_prox.STL
- added link l_middle_dist, mass 0.011; collision mesh filename=../meshes/l_middle_dist.STL; visual mesh filename=../meshes/l_middle_dist.STL
- added link l_middle_prox, mass 0.011; collision mesh filename=../meshes/l_middle_prox.STL; visual mesh filename=../meshes/l_middle_prox.STL
- added link l_palm, mass 0.427; collision mesh filename=../meshes/l_palm.STL; visual mesh filename=../meshes/l_palm.STL
- added link l_ring_dist, mass 0.008; collision mesh filename=../meshes/l_ring_dist.STL; visual mesh filename=../meshes/l_ring_dist.STL
- added link l_ring_prox, mass 0.011; collision mesh filename=../meshes/l_ring_prox.STL; visual mesh filename=../meshes/l_ring_prox.STL
- added link l_thumb_dist, mass 0.04; collision mesh filename=../meshes/l_thumb_dist.STL; visual mesh filename=../meshes/l_thumb_dist.STL
- added link l_thumb_prox, mass 0.005; collision mesh filename=../meshes/l_thumb_prox.STL; visual mesh filename=../meshes/l_thumb_prox.STL
- added link r_index_dist, mass 0.011; collision mesh filename=../meshes/r_index_dist.STL; visual mesh filename=../meshes/r_index_dist.STL
- added link r_index_prox, mass 0.008; collision mesh filename=../meshes/r_index_prox.STL; visual mesh filename=../meshes/r_index_prox.STL
- added link r_little_dist, mass 0.008; collision mesh filename=../meshes/r_little_dist.STL; visual mesh filename=../meshes/r_little_dist.STL
- added link r_little_prox, mass 0.008; collision mesh filename=../meshes/r_little_prox.STL; visual mesh filename=../meshes/r_little_prox.STL
- added link r_middle_dist, mass 0.011; collision mesh filename=../meshes/r_middle_dist.STL; visual mesh filename=../meshes/r_middle_dist.STL
- added link r_middle_prox, mass 0.011; collision mesh filename=../meshes/r_middle_prox.STL; visual mesh filename=../meshes/r_middle_prox.STL
- added link r_palm, mass 0.427; collision mesh filename=../meshes/r_palm.STL; visual mesh filename=../meshes/r_palm.STL
- added link r_ring_dist, mass 0.008; collision mesh filename=../meshes/r_ring_dist.STL; visual mesh filename=../meshes/r_ring_dist.STL
- added link r_ring_prox, mass 0.011; collision mesh filename=../meshes/r_ring_prox.STL; visual mesh filename=../meshes/r_ring_prox.STL
- added link r_thumb_dist, mass 0.04; collision mesh filename=../meshes/r_thumb_dist.STL; visual mesh filename=../meshes/r_thumb_dist.STL
- added link r_thumb_prox, mass 0.005; collision mesh filename=../meshes/r_thumb_prox.STL; visual mesh filename=../meshes/r_thumb_prox.STL
- link zarm_l7_link: geometry collision box size=0.08 0.05 0.16; collision cylinder length=0.08 radius=0.01
- link zarm_r7_link: geometry collision box size=0.08 0.05 0.16; collision cylinder length=0.08 radius=0.01
Joints:
- added joint l_indexMCP: type revolute, parent l_palm, child l_index_prox, origin xyz=-0.029003 0.088291 0.0022155 rpy=-0.029415 0.05236 0.034907, axis 1 0 0, limit lower=0 upper=1.309 effort=1.0 velocity=5.0
- added joint l_indexPIP: type revolute, parent l_index_prox, child l_index_dist, origin xyz=0 0.035 0 rpy=0.19353 0 0, axis 1 0 0, limit lower=0 upper=1.25 effort=1.0 velocity=5.0
- added joint l_littleMCP: type revolute, parent l_palm, child l_little_prox, origin xyz=0.033731 0.083777 0.0022155 rpy=-0.024909 -0.05236 -0.069813, axis 1 0 0, limit lower=0 upper=1.309 effort=1.0 velocity=5.0
- added joint l_littlePIP: type revolute, parent l_little_prox, child l_little_dist, origin xyz=0 0.035 0 rpy=0.20294 0 0, axis 1 0 0, limit lower=0 upper=1.25 effort=1.0 velocity=5.0
- added joint l_middleMCP: type revolute, parent l_palm, child l_middle_prox, origin xyz=-0.008 0.092284 -0.0017707 rpy=0 0 0, axis 1 0 0, limit lower=0 upper=1.309 effort=1.0 velocity=5.0
- added joint l_middlePIP: type revolute, parent l_middle_prox, child l_middle_dist, origin xyz=0 0.042 0 rpy=0.18357 0 0, axis 1 0 0, limit lower=0 upper=1.25 effort=1.0 velocity=5.0
- added joint l_palm_fixed_joint: type fixed, parent zarm_l7_link, child l_palm, origin xyz=0 0 -0.07 rpy=-1.57 0 -3.14
- added joint l_ringMCP: type revolute, parent l_palm, child l_ring_prox, origin xyz=0.013103 0.090291 -0.0017845 rpy=-0.0092374 -0.05236 -0.034907, axis 1 0 0, limit lower=0 upper=1.309 effort=1.0 velocity=5.0
- added joint l_ringPIP: type revolute, parent l_ring_prox, child l_ring_dist, origin xyz=0 0.042 0 rpy=0.16583 0 0, axis 1 0 0, limit lower=0 upper=1.25 effort=1.0 velocity=5.0
- added joint l_thumbCMC: type revolute, parent l_palm, child l_thumb_prox, origin xyz=-0.0245 0.022632 0.023263 rpy=0.14578 -1.0699 -0.12808, axis 0 1 0, limit lower=0 upper=1.5708 effort=1.0 velocity=5.0
- added joint l_thumbMCP: type revolute, parent l_thumb_prox, child l_thumb_dist, origin xyz=0 0 0.013647 rpy=0.87266 -0.49642 0, axis -1 0 0, limit lower=0 upper=0.8727 effort=1.0 velocity=5.0
- added joint r_indexMCP: type revolute, parent r_palm, child r_index_prox, origin xyz=0.029003 0.088231 -0.0039488 rpy=-0.09929 -0.054667 -0.031168, axis 1 0 0, limit lower=0 upper=1.309 effort=1.0 velocity=5.0
- added joint r_indexPIP: type revolute, parent r_index_prox, child r_index_dist, origin xyz=0 0.035 0 rpy=0.19353 0 0, axis 1 0 0, limit lower=0 upper=1.25 effort=1.0 velocity=5.0
- added joint r_littleMCP: type revolute, parent r_palm, child r_little_prox, origin xyz=-0.033731 0.083727 -0.0036339 rpy=-0.094666 0.057099 0.065996, axis 1 0 0, limit lower=0 upper=1.309 effort=1.0 velocity=5.0
- added joint r_littlePIP: type revolute, parent r_little_prox, child r_little_dist, origin xyz=0 0.035 0 rpy=0.20294 0 0, axis 1 0 0, limit lower=0 upper=1.25 effort=1.0 velocity=5.0
- added joint r_middleMCP: type revolute, parent r_palm, child r_middle_prox, origin xyz=0.008 0.091935 -0.0082038 rpy=-0.069813 0 0, axis 1 0 0, limit lower=0 upper=1.309 effort=1.0 velocity=5.0
- added joint r_middlePIP: type revolute, parent r_middle_prox, child r_middle_dist, origin xyz=0 0.042 0 rpy=0.18357 0 0, axis 1 0 0, limit lower=0 upper=1.25 effort=1.0 velocity=5.0
- added joint r_palm_fixed_joint: type fixed, parent zarm_r7_link, child r_palm, origin xyz=0 0 -0.07 rpy=-1.57 0 0
- added joint r_ringMCP: type revolute, parent r_palm, child r_ring_prox, origin xyz=-0.013103 0.089947 -0.0080786 rpy=-0.079113 0.054667 0.031168, axis 1 0 0, limit lower=0 upper=1.309 effort=1.0 velocity=5.0
- added joint r_ringPIP: type revolute, parent r_ring_prox, child r_ring_dist, origin xyz=0 0.042 0 rpy=0.16583 0 0, axis 1 0 0, limit lower=0 upper=1.25 effort=1.0 velocity=5.0
- added joint r_thumbCMC: type revolute, parent r_palm, child r_thumb_prox, origin xyz=0.0245 0.0242 0.021628 rpy=0 -0.49642 0, axis 0 -1 0, limit lower=0 upper=1.5708 effort=1.0 velocity=5.0
- added joint r_thumbMCP: type revolute, parent r_thumb_prox, child r_thumb_dist, origin xyz=0.013647 0 0 rpy=-0.39332 0.31115 -0.93514, axis 0 0 1, limit lower=0 upper=0.87266 effort=1.0 velocity=5.0
- joint zarm_l7_end_effector_joint: origin xyz=0 0.0 -0.17 rpy=0 3.14159265359 0 -> xyz=0 0.0 -0.17 rpy=0 0 0
- joint zarm_r7_end_effector_joint: origin xyz=0 0.0 -0.17 rpy=0 3.14159265359 0 -> xyz=0 0.0 -0.17 rpy=0 0 0
