Commit message: Add shared gravity compensation and 1 kg Leju claws

File: src/kuavo_isaaclab_scene/assets/kuavo_s63_twofinger/urdf/kuavo_s63_twofinger.urdf (robot description, URDF)
Before this commit: robot kuavo_s63_twofinger, 64 links, 63 joints
Links:
- link l_b_bar_1: mass 0.003 -> 0.004054054054054053
- link l_b_bar_2: mass 0.005 -> 0.006756756756756755
- link l_b_bar_3: mass 0.01 -> 0.01351351351351351
- link l_b_bar_4: mass 0.025 -> 0.03378378378378378
- link l_b_finger: mass 0.04 -> 0.05405405405405404
- link l_d405_camera: mass 0.001 -> 0.0013513513513513512
- link l_d405_camera_base: mass 0.072 -> 0.09729729729729727
- link l_d405_camera_connect: mass 0.001 -> 0.0013513513513513512
- link l_f_bar_1: mass 0.003 -> 0.004054054054054053
- link l_f_bar_2: mass 0.005 -> 0.006756756756756755
- link l_f_bar_3: mass 0.01 -> 0.01351351351351351
- link l_f_bar_4: mass 0.025 -> 0.03378378378378378
- link l_f_finger: mass 0.04 -> 0.05405405405405404
- link l_twofinger_base: mass 0.5 -> 0.6756756756756755
- link r_b_bar_1: mass 0.003 -> 0.004054054054054053
- link r_b_bar_2: mass 0.005 -> 0.006756756756756755
- link r_b_bar_3: mass 0.01 -> 0.01351351351351351
- link r_b_bar_4: mass 0.025 -> 0.03378378378378378
- link r_b_finger: mass 0.04 -> 0.05405405405405404
- link r_d405_camera: mass 0.001 -> 0.0013513513513513512
- link r_d405_camera_base: mass 0.072 -> 0.09729729729729727
- link r_d405_camera_connect: mass 0.001 -> 0.0013513513513513512
- link r_f_bar_1: mass 0.003 -> 0.004054054054054053
- link r_f_bar_2: mass 0.005 -> 0.006756756756756755
- link r_f_bar_3: mass 0.01 -> 0.01351351351351351
- link r_f_bar_4: mass 0.025 -> 0.03378378378378378
- link r_f_finger: mass 0.04 -> 0.05405405405405404
- link r_twofinger_base: mass 0.5 -> 0.6756756756756755

File: src/kuavo_isaaclab_scene/assets/leju_claw_two_finger/urdf/leju_claw_left.urdf (robot description, URDF)
Before this commit: robot leju_claw_left, 14 links, 13 joints
Links:
- link l_b_bar_1: mass 0.003 -> 0.004054054054054053
- link l_b_bar_2: mass 0.005 -> 0.006756756756756755
- link l_b_bar_3: mass 0.01 -> 0.01351351351351351
- link l_b_bar_4: mass 0.025 -> 0.03378378378378378
- link l_b_finger: mass 0.04 -> 0.05405405405405404
- link l_d405_camera: mass 0.001 -> 0.0013513513513513512
- link l_d405_camera_base: mass 0.072 -> 0.09729729729729727
- link l_d405_camera_connect: mass 0.001 -> 0.0013513513513513512
- link l_f_bar_1: mass 0.003 -> 0.004054054054054053
- link l_f_bar_2: mass 0.005 -> 0.006756756756756755
- link l_f_bar_3: mass 0.01 -> 0.01351351351351351
- link l_f_bar_4: mass 0.025 -> 0.03378378378378378
- link l_f_finger: mass 0.04 -> 0.05405405405405404
- link l_twofinger_base: mass 0.5 -> 0.6756756756756755

File: src/kuavo_isaaclab_scene/assets/leju_claw_two_finger/urdf/leju_claw_right.urdf (robot description, URDF)
Before this commit: robot leju_claw_right, 14 links, 13 joints
Links:
- link r_b_bar_1: mass 0.003 -> 0.004054054054054053
- link r_b_bar_2: mass 0.005 -> 0.006756756756756755
- link r_b_bar_3: mass 0.01 -> 0.01351351351351351
- link r_b_bar_4: mass 0.025 -> 0.03378378378378378
- link r_b_finger: mass 0.04 -> 0.05405405405405404
- link r_d405_camera: mass 0.001 -> 0.0013513513513513512
- link r_d405_camera_base: mass 0.072 -> 0.09729729729729727
- link r_d405_camera_connect: mass 0.001 -> 0.0013513513513513512
- link r_f_bar_1: mass 0.003 -> 0.004054054054054053
- link r_f_bar_2: mass 0.005 -> 0.006756756756756755
- link r_f_bar_3: mass 0.01 -> 0.01351351351351351
- link r_f_bar_4: mass 0.025 -> 0.03378378378378378
- link r_f_finger: mass 0.04 -> 0.05405405405405404
- link r_twofinger_base: mass 0.5 -> 0.6756756756756755

Commit message: Remove duplicate S63 wrist camera mounts from Leju variant

File: src/kuavo_isaaclab_scene/assets/kuavo_s63_twofinger/urdf/kuavo_s63_twofinger.urdf (robot description, URDF)
Before this commit: robot kuavo_s63_twofinger, 64 links, 63 joints
Links:
- link zarm_l7_link: geometry collision cylinder length=0.14 radius=0.04; visual mesh filename=../meshes/l_hand_pitch_wrist_only.STL
- link zarm_r7_link: geometry collision cylinder length=0.14 radius=0.04; visual mesh filename=../meshes/r_hand_pitch_wrist_only.STL
