Commit message: Restore official S63 assets and add reusable Leju two-finger claw variant

File: src/kuavo_isaaclab_scene/assets/kuavo_s63/urdf/kuavo_s63.urdf (robot description, URDF)
Before this commit: robot biped_s63, 36 links, 35 joints
Links:
- link zarm_l7_link: geometry collision cylinder length=0.14 radius=0.04; visual mesh filename=../meshes/l_hand_pitch_noHand.STL
- link zarm_r7_link: geometry collision cylinder length=0.14 radius=0.04; visual mesh filename=../meshes/r_hand_pitch_noHand.STL
Joints:
- joint zarm_l7_end_effector_joint: origin xyz=0.135599 -0.017281 -0.115070 rpy=2.779374508 -0.751879414 0.253261563 -> xyz=0 0.0 -0.17 rpy=0 0 0
- joint zarm_r7_end_effector_joint: origin xyz=0.135599 0.017281 -0.115070 rpy=-2.779374508 -0.751879414 -0.253261563 -> xyz=0 0.0 -0.17 rpy=0 0 0

Commit message: Calibrate S63 simulation control and tooling

File: src/kuavo_isaaclab_scene/assets/kuavo_s63/urdf/kuavo_s63.urdf (robot description, URDF)
Before this commit: robot biped_s63, 36 links, 35 joints
Links:
- link zarm_l7_link: geometry collision cylinder length=0.14 radius=0.04; visual mesh filename=../meshes/l_hand_pitch.STL
- link zarm_r7_link: geometry collision cylinder length=0.14 radius=0.04; visual mesh filename=../meshes/r_hand_pitch.STL
