Commit message: Fix S56 and S200062 four-bar gripper closure
Restore passive central links and physical finger-to-bar hinges, validate reset and contact motion, and document the post-fix checkpoint-40K evaluation and remaining limitations.

File: src/kuavo_isaaclab_scene/assets/kuavo_s200062/urdf/biped_s200062.urdf (robot description, URDF)
Before this commit: robot biped_s200062, 64 links, 63 joints
Joints:
- joint l_b_bar_4_joint: axis (none) -> 0 1 0; limit (none) -> lower=-0.698 upper=0.698 effort=5 velocity=5; type fixed -> revolute
- joint l_f_bar_4_joint: axis (none) -> 0 1 0; limit (none) -> lower=-0.698 upper=0.698 effort=5 velocity=5; type fixed -> revolute
- joint r_b_bar_4_joint: axis (none) -> 0 1 0; limit (none) -> lower=-0.698 upper=0.698 effort=5 velocity=5; type fixed -> revolute
- joint r_f_bar_4_joint: axis (none) -> 0 1 0; limit (none) -> lower=-0.698 upper=0.698 effort=5 velocity=5; type fixed -> revolute

File: src/kuavo_isaaclab_scene/assets/kuavo_s56/urdf/kuavo_s56_twofinger.urdf (robot description, URDF)
Before this commit: robot kuavo_s56_twofinger, 82 links, 81 joints
Joints:
- joint l_b_bar_4_joint: axis (none) -> 0 1 0; limit (none) -> lower=-0.698 upper=0.698 effort=5 velocity=5; type fixed -> revolute
- joint l_f_bar_4_joint: axis (none) -> 0 1 0; limit (none) -> lower=-0.698 upper=0.698 effort=5 velocity=5; type fixed -> revolute
- joint r_b_bar_4_joint: axis (none) -> 0 1 0; limit (none) -> lower=-0.698 upper=0.698 effort=5 velocity=5; type fixed -> revolute
- joint r_f_bar_4_joint: axis (none) -> 0 1 0; limit (none) -> lower=-0.698 upper=0.698 effort=5 velocity=5; type fixed -> revolute

Commit message: Preserve local Task1 planning, replay, and S200062 asset changes

File: src/kuavo_isaaclab_scene/assets/kuavo_s200062/urdf/biped_s200062.urdf (robot description, URDF)
Before this commit: robot biped_s200062, 64 links, 63 joints
Joints:
- joint zarm_l7_end_effector_1_joint: origin xyz=0 0.0 -0.08 rpy=0 0 0 -> xyz=0 0.0 -0.13 rpy=0 0 0
- joint zarm_l7_end_effector_2_joint: origin xyz=0.03 0.0 -0.17 rpy=0 0 0 -> xyz=0.03 0.0 -0.22 rpy=0 0 0
- joint zarm_l7_end_effector_joint: origin xyz=0 0.0 -0.17 rpy=0 0 0 -> xyz=0 0.0 -0.22 rpy=0 0 0
- joint zarm_r7_end_effector_1_joint: origin xyz=0 0.0 -0.08 rpy=0 0 0 -> xyz=0 0.0 -0.13 rpy=0 0 0
- joint zarm_r7_end_effector_2_joint: origin xyz=0.03 0.0 -0.17 rpy=0 0 0 -> xyz=0.03 0.0 -0.22 rpy=0 0 0
- joint zarm_r7_end_effector_joint: origin xyz=0 0.0 -0.17 rpy=0 0 0 -> xyz=0 0.0 -0.22 rpy=0 0 0
